Commit message: Added nav2_params_custom into nav2_bringup in order to change robot model and configs from differential to omnidirectional

File: ros_2_ws/src/octobot_2/install/octobot_2/share/octobot_2/urdf/NuevaBaseMetal2.urdf (robot description, URDF)
Before this commit: robot Octobot_2, 8 links, 7 joints
Links:
- added link imu_link
Joints:
- added joint imu_joint: type fixed, parent base_link, child imu_link, origin xyz=0.0 0 0.0 rpy=0 0 0, axis 1 0 0

Commit message: Quickfix xdxdxdxd!

File: ros_2_ws/src/octobot_2/install/octobot_2/share/octobot_2/urdf/NuevaBaseMetal2.urdf (robot description, URDF)
Before this commit: robot octobot_2, 7 links, 6 joints
Links:
- removed link BL_link
- removed link BR_link
- removed link Base_link
- removed link Camera_link
- removed link FL_link
- removed link FR_link
- removed link Lidar_link
- added link BL_Link, mass 0.088298; collision mesh filename=package://octobot_2/meshes/BL_Link.STL; visual mesh filename=package://octobot_2/meshes/BL_Link.STL
- added link BR_Link, mass 0.088298; collision mesh filename=package://octobot_2/meshes/BR_Link.STL; visual mesh filename=package://octobot_2/meshes/BR_Link.STL
- added link Camera_Link, mass 0.15394; collision mesh filename=package://octobot_2/meshes/Camera_Link.STL; visual mesh filename=package://octobot_2/meshes/Camera_Link.STL
- added link FL_Link, mass 0.088298; collision mesh filename=package://octobot_2/meshes/FL_Link.STL; visual mesh filename=package://octobot_2/meshes/FL_Link.STL
- added link FR_Link, mass 0.088298; collision mesh filename=package://octobot_2/meshes/FR_Link.STL; visual mesh filename=package://octobot_2/meshes/FR_Link.STL
- added link Lidar_Link, mass 0.15394; collision mesh filename=package://octobot_2/meshes/Lidar_Link.STL; visual mesh filename=package://octobot_2/meshes/Lidar_Link.STL
- added link base_footprint
- added link base_link, mass 1.1176; collision mesh filename=package://octobot_2/meshes/Base_link.STL; visual mesh filename=package://octobot_2/meshes/Base_link.STL
- added link imu_link
Joints:
- removed joint BL_joint
- removed joint BR_joint
- removed joint FL_joint
- removed joint FR_joint
- removed joint cam_joint
- removed joint lidar_joint
- added joint BL_Joint: type continuous, parent base_link, child BL_Link, origin xyz=-0.20406 0.20406 0.018501 rpy=1.5708 0 -2.3562, axis 0 0 -1
- added joint BR_Joint: type continuous, parent base_link, child BR_Link, origin xyz=-0.20406 -0.20406 0.0185 rpy=1.5708 0 -0.7854, axis 0 0 -1
- added joint Base_footprint_joint: type fixed, parent base_link, child base_footprint, origin xyz=0 0 0 rpy=0 0 0
- added joint Camera_Joint: type fixed, parent base_link, child Camera_Link, origin xyz=0 0 0 rpy=0 0 0, axis 0 0 0.063
- added joint FL_Joint: type continuous, parent base_link, child FL_Link, origin xyz=0.20406 0.20406 0.018501 rpy=1.5708 0 2.3562, axis 0 0 -1
- added joint FR_Joint: type continuous, parent base_link, child FR_Link, origin xyz=0.20406 -0.20406 0.0185 rpy=1.5708 0 0.7854, axis 0 0 -1
- added joint Lidar_Joint: type fixed, parent base_link, child Lidar_Link, origin xyz=0 0 0 rpy=0 0 0, axis 0 0 0
- added joint imu_joint: type fixed, parent base_link, child imu_link, origin xyz=0.0 0 0.0 rpy=0 0 0, axis 1 0 0

File: ros_2_ws/src/octobot_2/install/octobot_2/share/octobot_2/urdf/NuevaBaseMetal3.urdf (robot description, URDF)
Before this commit: robot octobot_2, 8 links, 7 joints
Links:
- removed link cam_link
Joints:
- removed joint cam_joint
