Commit message: first version with navigation

File: ros_1_ws/src/NuevaBaseMetal3/urdf/NuevaBaseMetal3.urdf (robot description, URDF)
Before this commit: robot octobot_2, 7 links, 6 joints
Links:
- link base_link: geometry collision mesh filename=package://NuevaBaseMetal3/meshes/base_link.STL; visual mesh filename=package://NuevaBaseMetal3/meshes/base_link.STL
- link bl_link: geometry collision mesh filename=package://NuevaBaseMetal3/meshes/bl_link.STL; visual mesh filename=package://NuevaBaseMetal3/meshes/bl_link.STL
- link br_link: geometry collision mesh filename=package://NuevaBaseMetal3/meshes/br_link.STL; visual mesh filename=package://NuevaBaseMetal3/meshes/br_link.STL
- link fl_link: geometry collision mesh filename=package://NuevaBaseMetal3/meshes/fl_link.STL; visual mesh filename=package://NuevaBaseMetal3/meshes/fl_link.STL
- link fr_link: geometry collision mesh filename=package://NuevaBaseMetal3/meshes/fr_link.STL; visual mesh filename=package://NuevaBaseMetal3/meshes/fr_link.STL
- link lidar_link: geometry collision mesh filename=package://NuevaBaseMetal3/meshes/lidar_link.STL; visual mesh filename=package://NuevaBaseMetal3/meshes/lidar_link.STL
